File: PCB/Ogen.kicad_pcb (KiCad board)
At the start: 2 copper layers, 28 x 21.5 mm, 17 parts, among them J1 Input, U1 PMW3360DM-T2QU, U2 TLV70019, U3 TXS0102DCU, U4 TXS0102DCU, U5 TXS0102DCU

Commit message: ✨ ♻️ - Add metadata required to generate BOM and POS files for JLCPCB SMT assembly service (can use Fabrication Toolkit plugin to generate up to date BOM and POS). Add description to PCB and schema files. Replace TLV70019 (rupture) part by VRH1902LTX (in stock).
Parts:
- U2: value TLV70019 -> VRH1902LTX
Other:
- board text added: "Ogen V1.2"
- board text removed: "Ogen V1.1"
Changed lines of the file:
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@@
   )
   (paper "A4")
+  (title_block
+    (title "Ogen")
+    (date "2022-11-11")
+    (rev "V1.2")
+    (company "Ariamelon")
+  )
   (layers
     (0 "F.Cu" signal)
@@
       (plotinvisibletext false)
       (sketchpadsonfab false)
-      (subtractmaskfromsilk false)
+      (subtractmaskfromsilk true)
       (outputformat 1)
       (mirror false)
       (drillshape 0)
       (scaleselection 1)
-      (outputdirectory "OgenV1.1-Gerbers")
+      (outputdirectory "data/production/gerber/")
     )
   )
@@
     (property "Sheetfile" "Ogen.kicad_sch")
     (property "Sheetname" "")
-    (attr through_hole)
+    (property "exclude_from_bom" "")
+    (attr through_hole exclude_from_bom)
     (fp_text reference "J1" (at 0 -10.822 unlocked) (layer "F.SilkS")
       (effects (font (size 0.75 0.75) (thickness 0.125)))
@@
     (at 26.572 23.734 90)
     (tags "DIP 18 Pixart PMW3360 PMW3360DM-T2QU optical mouse sensor")
-    (property "Sheetfile" "Ogen.kicad_sch")
-    (property "Sheetname" "")
-    (attr through_hole)
+    (property "LCSC Part #" "")
+    (property "Sheetfile" "Ogen.kicad_sch")
+    (property "Sheetname" "")
+    (attr through_hole exclude_from_pos_files)
     (fp_text reference "U1" (at 4.984 -7.822 unlocked) (layer "F.SilkS")
       (effects (font (size 0.75 0.75) (thickness 0.125)))
@@
     (property "Sheetfile" "Ogen.kicad_sch")
     (property "Sheetname" "")
+    (property "exclude_from_bom" "")
     (clearance 1.8)
-    (attr exclude_from_pos_files)
+    (attr exclude_from_pos_files exclude_from_bom)
     (fp_text reference "H1" (at 0 -3.2 -90 unlocked) (layer "F.SilkS") hide
       (effects (font (size 0.75 0.75) (thickness 0.125)))
@@
     (property "Sheetfile" "Ogen.kicad_sch")
     (property "Sheetname" "")
+    (property "exclude_from_bom" "")
     (clearance 1.8)
-    (attr exclude_from_pos_files)
+    (attr exclude_from_pos_files exclude_from_bom)
     (fp_text reference "H2" (at 0 -3.2 -90 unlocked) (layer "F.SilkS") hide
       (effects (font (size 0.75 0.75) (thickness 0.125)))
@@
     (descr "VSSOP-8 2.3x2mm Pitch 0.5mm")
     (tags "VSSOP-8 2.3x2mm Pitch 0.5mm")
+    (property "JLCPCB Rotation Offset" "180")
+    (property "LCSC Part #" "C9382C53434")
     (property "Sheetfile" "Ogen.kicad_sch")
     (property "Sheetname" "")
@@
     (descr "Capacitor SMD 0603 (1608 Metric), square (rectangular) end terminal, IPC_7351 nominal, (Body size source: IPC-SM-782 page 76, https://www.pcb-3d.com/wordpress/wp-content/uploads/ipc-sm-782a_amendment_1_and_2.pdf), generated with kicad-footprint-generator")
     (tags "capacitor")
+    (property "LCSC Part #" "C19666")
     (property "Sheetfile" "Ogen.kicad_sch")
     (property "Sheetname" "")
@@
     (descr "VSSOP-8 2.3x2mm Pitch 0.5mm")
     (tags "VSSOP-8 2.3x2mm Pitch 0.5mm")
+    (property "JLCPCB Rotation Offset" "180")
+    (property "LCSC Part #" "C53434")
     (property "Sheetfile" "Ogen.kicad_sch")
     (property "Sheetname" "")
@@
     (descr "Capacitor SMD 0603 (1608 Metric), square (rectangular) end terminal, IPC_7351 nominal, (Body size source: IPC-SM-782 page 76, https://www.pcb-3d.com/wordpress/wp-content/uploads/ipc-sm-782a_amendment_1_and_2.pdf), generated with kicad-footprint-generator")
     (tags "capacitor")
+    (property "LCSC Part #" "C15849")
     (property "Sheetfile" "Ogen.kicad_sch")
     (property "Sheetname" "")
@@
     (descr "Resistor SMD 0603 (1608 Metric), square (rectangular) end terminal, IPC_7351 nominal, (Body size source: IPC-SM-782 page 72, https://www.pcb-3d.com/wordpress/wp-content/uploads/ipc-sm-782a_amendment_1_and_2.pdf), generated with kicad-footprint-generator")
     (tags "resistor")
+    (property "LCSC Part #" "C25804")
     (property "Sheetfile" "Ogen.kicad_sch")
     (property "Sheetname" "")
@@
     (descr "Capacitor SMD 0603 (1608 Metric), square (rectangular) end terminal, IPC_7351 nominal, (Body size source: IPC-SM-782 page 76, https://www.pcb-3d.com/wordpress/wp-content/uploads/ipc-sm-782a_amendment_1_and_2.pdf), generated with kicad-footprint-generator")
     (tags "capacitor")
+    (property "LCSC Part #" "C14663")
     (property "Sheetfile" "Ogen.kicad_sch")
     (property "Sheetname" "")
@@
     (descr "Resistor SMD 0603 (1608 Metric), square (rectangular) end terminal, IPC_7351 nominal, (Body size source: IPC-SM-782 page 72, https://www.pcb-3d.com/wordpress/wp-content/uploads/ipc-sm-782a_amendment_1_and_2.pdf), generated with kicad-footprint-generator")
     (tags "resistor")
+    (property "LCSC Part #" "C227492")
     (property "Sheetfile" "Ogen.kicad_sch")
     (property "Sheetname" "")
@@
     (property "Sheetfile" "Ogen.kicad_sch")
     (property "Sheetname" "")
-    (attr exclude_from_pos_files)
+    (property "exclude_from_bom" "")
+    (attr exclude_from_pos_files exclude_from_bom)
     (fp_text reference "JP1" (at -2.678 0 unlocked) (layer "F.SilkS")
       (effects (font (size 0.75 0.75) (thickness 0.125)))
@@
     (descr "SOT, 5 Pin (https://www.jedec.org/sites/default/files/docs/Mo-178c.PDF variant AA), generated with kicad-footprint-generator ipc_gullwing_generator.py")
     (tags "SOT TO_SOT_SMD")
+    (property "JLCPCB Rotation Offset" "-90")
+    (property "LCSC Part #" "C697975")
     (property "Sheetfile" "Ogen.kicad_sch")
     (property "Sheetname" "")
@@
       (effects (font (size 0.75 0.75) (thickness 0.125)))
     )
-    (fp_text value "TLV70019" (at 0 2.4 -90 unlocked) (layer "F.Fab")
+    (fp_text value "VRH1902LTX" (at 0 2.4 -90 unlocked) (layer "F.Fab")
       (effects (font (size 1 1) (thickness 0.15)))
     )
@@
     (descr "VSSOP-8 2.3x2mm Pitch 0.5mm")
     (tags "VSSOP-8 2.3x2mm Pitch 0.5mm")
+    (property "JLCPCB Rotation Offset" "180")
+    (property "LCSC Part #" "C53434")
     (property "Sheetfile" "Ogen.kicad_sch")
     (property "Sheetname" "")
@@
     (descr "Capacitor SMD 0603 (1608 Metric), square (rectangular) end terminal, IPC_7351 nominal, (Body size source: IPC-SM-782 page 76, https://www.pcb-3d.com/wordpress/wp-content/uploads/ipc-sm-782a_amendment_1_and_2.pdf), generated with kicad-footprint-generator")
     (tags "capacitor")
+    (property "LCSC Part #" "C15849")
     (property "Sheetfile" "Ogen.kicad_sch")
     (property "Sheetname" "")
@@
     (descr "Resistor SMD 0603 (1608 Metric), square (rectangular) end terminal, IPC_7351 nominal, (Body size source: IPC-SM-782 page 72, https://www.pcb-3d.com/wordpress/wp-content/uploads/ipc-sm-782a_amendment_1_and_2.pdf), generated with kicad-footprint-generator")
     (tags "resistor")
+    (property "LCSC Part #" "C25804")
     (property "Sheetfile" "Ogen.kicad_sch")
     (property "Sheetname" "")
@@
     (property "Sheetfile" "Ogen.kicad_sch")
     (property "Sheetname" "")
-    (attr board_only exclude_from_pos_files)
+    (property "exclude_from_bom" "")
+    (attr board_only exclude_from_pos_files exclude_from_bom)
     (fp_text reference "A1" (at 0 0) (layer "B.SilkS") hide
       (effects (font (size 1.524 1.524) (thickness 0.3)) (justify mirror))
@@
     (effects (font (size 0.75 0.75) (thickness 0.125)) (justify mirror))
   )
-  (gr_text "Ogen V1.1" (at 27.334 16.674) (layer "B.SilkS")
+  (gr_text "Ogen V1.2" (at 27.334 16.674) (layer "B.SilkS")
     (effects (font (size 0.75 0.75) (thickness 0.125)) (justify mirror))
   )
